File: C# Based Smart Gardener  Final PCB/C# Based Smart Gardener.kicad_pcb (KiCad board)
At the start: 2 copper layers, 79.2 x 96.3 mm, 44 parts, among them J1 HEATER, J10 LDR, J11 TEMPERATURE, J12 HUMIDITY, J2 LAMP, J3 PUMP1, J4 FAN, J5 PUMP2, J6 12V, J9 HC-05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

Commit message: PCB Update
Parts:
- added G***: LOGO, xdxd:rtrt, F.Cu at (138.6, 87.4)
- J6: value 12V -> 12V
- R10: value 2.2k -> 220
- moved D1 14.3 mm to (171.7, 71.9), turned to 90 degrees
- moved C7 7.67 mm to (171.7, 95.1)
- moved D2 7.29 mm to (185.8, 89.3), turned to 180 degrees
- moved U3 4.71 mm to (184.5, 97.7), turned to 0 degrees
- moved C8 4.70 mm to (166.8, 95.1)
- moved U1 3.67 mm to (184.4, 82.8)
- moved R9 1.97 mm to (176.4, 108.8)
- moved R8 1.51 mm to (171.7, 101.8)
- moved C2 0.76 mm to (171.7, 78.4)
- moved C3 0.76 mm to (171.7, 86.8)
- moved C4 0.71 mm to (166.8, 86.8)
- moved C1 0.71 mm to (166.8, 78.4)
- moved C5 0.42 mm to (183.8, 112.0)
- moved C6 0.26 mm to (185.3, 106.6)
Routing:
- net +12V: track 276.6 -> 305.0 mm, vias 1 -> 2
- net GND: track 83.3 -> 110.2 mm, vias 12 -> 9
- net +3V3: track 63.9 -> 84.7 mm
- net Net-(C5-Pad1): track 20.9 -> 38.4 mm
- net Net-(R8-Pad1): track 14.4 -> 26.0 mm
- net +5V: track 163.5 -> 174.6 mm, vias 4 -> 2
- net Net-(C1-Pad1): track 20.0 -> 25.7 mm
- net Net-(J3-Pad1): track 24.8 -> 28.6 mm
- net Net-(J4-Pad1): track 24.8 -> 28.6 mm
- net Net-(J5-Pad1): track 25.0 -> 28.6 mm
- net Net-(J2-Pad1): track 24.8 -> 28.5 mm
- net SENSOR2: track 33.3 -> 31.9 mm, vias 2 -> 0
- net 2.1: track 19.4 -> 20.0 mm
- net RXD: track 25.4 -> 25.7 mm, vias 2 -> 0
- net SENSOR3: track 35.1 -> 35.0 mm, vias 1 -> 0
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Other:
- board text added: "vorun"

Commit message: Update PCB
Parts:
- removed G***: LOGO, xdxd:rtrt
- added J7: HC-05 3D, Connector_PinSocket_2.54mm:PinSocket_1x04_P2.54mm_Vertical, F.Cu at (126.0, 83.6)
- J6: value 12V -> 12V ADAPTOR
