File: C# Based Smart Gardener  Final PCB/C# Based Smart Gardener.kicad_pcb (KiCad board)
At the start: 2 copper layers, 79.2 x 114.6 mm, 51 parts, among them J1 HEATER, J10 LDR, J11 TEMPERATURE, J12 HUMIDITY, J2 PUMP1, J3 LAMP, J4 PUMP2, J5 FAN, J6 12V ADAPTOR, J7 HC-05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

Commit message: PCB Updated
Parts:
- Q1, Q2, Q3, Q4, Q5: value IRLZ44N -> 2SK3919; footprint Package_TO_SOT_SMD:TO-263-2 -> Package_TO_SOT_SMD:TO-252-2
- moved R1 1.05 mm to (156.2, 129.0)
- moved R2 1.02 mm to (141.6, 129.0)
- moved R3 1.02 mm to (185.4, 129.0)
- moved R4 1.02 mm to (170.7, 129.0)
- moved R6 1.02 mm to (127.0, 129.0)
- moved Q1 1.02 mm to (154.7, 147.3)
- moved Q2 1.02 mm to (140.1, 147.3)
- moved Q3 1.02 mm to (183.9, 147.3)
- moved Q4 1.02 mm to (169.3, 147.3)
- moved Q5 1.02 mm to (125.5, 147.3)
- moved R11 1.02 mm to (154.7, 135.3)
- moved R12 1.02 mm to (140.1, 135.3)
- moved R13 1.02 mm to (183.9, 135.3)
- moved R14 1.02 mm to (169.3, 135.3)
- moved R5 1.02 mm to (125.5, 135.3)
Routing:
- net Net-(Q2-Pad1): track 6.70 -> 13.1 mm
- net Net-(Q3-Pad1): track 11.4 -> 6.08 mm
- net Net-(Q5-Pad1): track 11.4 -> 13.1 mm
- net Net-(Q4-Pad1): track 11.4 -> 13.1 mm
- net Net-(Q1-Pad1): track 11.9 -> 13.1 mm
- net Net-(R3-Pad2): track 21.5 -> 22.5 mm
- net Net-(R1-Pad2): track 4.45 -> 5.38 mm
- net Net-(R6-Pad2): track 9.66 -> 10.5 mm
- net Net-(R4-Pad2): track 5.95 -> 6.81 mm
- net Net-(R2-Pad2): track 12.7 -> 13.5 mm
