File: C# Based Smart Gardener  Final PCB/C# Based Smart Gardener.sch (KiCad schematic (older format))
At the start: 44 parts, among them J1 HEATER, J10 LDR, J11 TEMPERATURE, J12 HUMIDITY, J2 LAMP, J3 PUMP1, J4 FAN, J5 PUMP2, J6 12V ADAPTOR, J9 HC-05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

Commit message: PCB Update
Parts:
- R10: value 2.2k -> 220
Changed lines of the file:
@@
 P 6850 1300
 F 0 "R10" H 6920 1346 50  0000 L CNN
-F 1 "2.2k" H 6920 1255 50  0000 L CNN
+F 1 "220" H 6920 1255 50  0000 L CNN
 F 2 "Resistor_THT:R_Axial_DIN0204_L3.6mm_D1.6mm_P5.08mm_Horizontal" V 6780 1300 50  0001 C CNN
 F 3 "~" H 6850 1300 50  0001 C CNN

Commit message: Update PCB
Parts:
- added J7: HC-05 3D, Connector_PinSocket_2.54mm:PinSocket_1x04_P2.54mm_Vertical, symbol Connector:Conn_01x04_Female
Changed lines of the file:
@@
 Wire Wire Line
 	1600 3050 2050 3050
+$Comp
+L Connector:Conn_01x04_Female J7
+U 1 1 62ACDE9B
+P 4750 3150
+F 0 "J7" H 4778 3126 50  0000 L CNN
+F 1 "HC-05 3D" H 4778 3035 50  0000 L CNN
+F 2 "Connector_PinSocket_2.54mm:PinSocket_1x04_P2.54mm_Vertical" H 4750 3150 50  0001 C CNN
+F 3 "~" H 4750 3150 50  0001 C CNN
+	1    4750 3150
+	1    0    0    -1
+$EndComp
 $EndSCHEMATC
