File: C# Based Smart Gardener  Final PCB/C# Based Smart Gardener.sch (KiCad schematic (older format))
At the start: 51 parts, among them J1 HEATER, J10 LDR, J11 TEMPERATURE, J12 HUMIDITY, J2 PUMP1, J3 LAMP, J4 PUMP2, J5 FAN, J6 12V ADAPTOR, J7 HC-05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

Commit message: PCB Updated
Parts:
- Q1, Q2, Q3, Q4, Q5: value IRLZ44N -> 2SK3919; footprint Package_TO_SOT_SMD:TO-263-2 -> Package_TO_SOT_SMD:TO-252-2
Changed lines of the file:
@@
 P 2200 6100
 F 0 "Q3" H 2404 6146 50  0000 L CNN
-F 1 "IRLZ44N" H 2404 6055 50  0000 L CNN
-F 2 "Package_TO_SOT_SMD:TO-263-2" H 2450 6025 50  0001 L CIN
+F 1 "2SK3919" H 2404 6055 50  0000 L CNN
+F 2 "Package_TO_SOT_SMD:TO-252-2" H 2450 6025 50  0001 L CIN
 F 3 "http://www.irf.com/product-info/datasheets/data/irlz44n.pdf" H 2200 6100 50  0001 L CNN
 	1    2200 6100
@@
 P 2150 3250
 F 0 "Q5" H 2354 3296 50  0000 L CNN
-F 1 "IRLZ44N" H 2354 3205 50  0000 L CNN
-F 2 "Package_TO_SOT_SMD:TO-263-2" H 2400 3175 50  0001 L CIN
+F 1 "2SK3919" H 2354 3205 50  0000 L CNN
+F 2 "Package_TO_SOT_SMD:TO-252-2" H 2400 3175 50  0001 L CIN
 F 3 "http://www.irf.com/product-info/datasheets/data/irlz44n.pdf" H 2150 3250 50  0001 L CNN
 	1    2150 3250
@@
 P 2200 7000
 F 0 "Q4" H 2404 7046 50  0000 L CNN
-F 1 "IRLZ44N" H 2404 6955 50  0000 L CNN
-F 2 "Package_TO_SOT_SMD:TO-263-2" H 2450 6925 50  0001 L CIN
+F 1 "2SK3919" H 2404 6955 50  0000 L CNN
+F 2 "Package_TO_SOT_SMD:TO-252-2" H 2450 6925 50  0001 L CIN
 F 3 "http://www.irf.com/product-info/datasheets/data/irlz44n.pdf" H 2200 7000 50  0001 L CNN
 	1    2200 7000
@@
 P 2200 5100
 F 0 "Q2" H 2404 5146 50  0000 L CNN
-F 1 "IRLZ44N" H 2404 5055 50  0000 L CNN
-F 2 "Package_TO_SOT_SMD:TO-263-2" H 2450 5025 50  0001 L CIN
+F 1 "2SK3919" H 2404 5055 50  0000 L CNN
+F 2 "Package_TO_SOT_SMD:TO-252-2" H 2450 5025 50  0001 L CIN
 F 3 "http://www.irf.com/product-info/datasheets/data/irlz44n.pdf" H 2200 5100 50  0001 L CNN
 	1    2200 5100
@@
 P 2200 4150
 F 0 "Q1" H 2404 4196 50  0000 L CNN
-F 1 "IRLZ44N" H 2404 4105 50  0000 L CNN
-F 2 "Package_TO_SOT_SMD:TO-263-2" H 2450 4075 50  0001 L CIN
+F 1 "2SK3919" H 2404 4105 50  0000 L CNN
+F 2 "Package_TO_SOT_SMD:TO-252-2" H 2450 4075 50  0001 L CIN
 F 3 "http://www.irf.com/product-info/datasheets/data/irlz44n.pdf" H 2200 4150 50  0001 L CNN
 	1    2200 4150
